Commit message: WIP Update: Melodic sub-workspace

File: src/fs_resources/barrett_hand_description/robots/bh_alone_v2.urdf (robot description, URDF)
Before this commit: robot bhand, 110 links, 109 joints
Links:
- removed link bh_link1_sensor10_link
- removed link bh_link1_sensor11_link
- removed link bh_link1_sensor12_link
- removed link bh_link1_sensor13_link
- removed link bh_link1_sensor14_link
- removed link bh_link1_sensor15_link
- removed link bh_link1_sensor16_link
- removed link bh_link1_sensor17_link
- removed link bh_link1_sensor18_link
- removed link bh_link1_sensor19_link
- removed link bh_link1_sensor1_link
- removed link bh_link1_sensor20_link
- removed link bh_link1_sensor21_link
- removed link bh_link1_sensor22_link
- removed link bh_link1_sensor23_link
- removed link bh_link1_sensor24_link
- removed link bh_link1_sensor2_link
- removed link bh_link1_sensor3_link
- removed link bh_link1_sensor4_link
- removed link bh_link1_sensor5_link
- removed link bh_link1_sensor6_link
- removed link bh_link1_sensor7_link
- removed link bh_link1_sensor8_link
- removed link bh_link1_sensor9_link
- removed link bh_link2_sensor10_link
- removed link bh_link2_sensor11_link
- removed link bh_link2_sensor12_link
- removed link bh_link2_sensor13_link
- removed link bh_link2_sensor14_link
- removed link bh_link2_sensor15_link
- removed link bh_link2_sensor16_link
- removed link bh_link2_sensor17_link
- removed link bh_link2_sensor18_link
- removed link bh_link2_sensor19_link
- removed link bh_link2_sensor1_link
- removed link bh_link2_sensor20_link
- removed link bh_link2_sensor21_link
- removed link bh_link2_sensor22_link
- removed link bh_link2_sensor23_link
- removed link bh_link2_sensor24_link
- removed link bh_link2_sensor2_link
- removed link bh_link2_sensor3_link
- removed link bh_link2_sensor4_link
- removed link bh_link2_sensor5_link
- removed link bh_link2_sensor6_link
- removed link bh_link2_sensor7_link
- removed link bh_link2_sensor8_link
- removed link bh_link2_sensor9_link
- removed link bh_link3_sensor10_link
- removed link bh_link3_sensor11_link
- removed link bh_link3_sensor12_link
- removed link bh_link3_sensor13_link
- removed link bh_link3_sensor14_link
- removed link bh_link3_sensor15_link
- removed link bh_link3_sensor16_link
- removed link bh_link3_sensor17_link
- removed link bh_link3_sensor18_link
- removed link bh_link3_sensor19_link
- removed link bh_link3_sensor1_link
- removed link bh_link3_sensor20_link
- removed link bh_link3_sensor21_link
- removed link bh_link3_sensor22_link
- removed link bh_link3_sensor23_link
- removed link bh_link3_sensor24_link
- removed link bh_link3_sensor2_link
- removed link bh_link3_sensor3_link
- removed link bh_link3_sensor4_link
- removed link bh_link3_sensor5_link
- removed link bh_link3_sensor6_link
- removed link bh_link3_sensor7_link
- removed link bh_link3_sensor8_link
- removed link bh_link3_sensor9_link
- removed link bh_palm_sensor_10_link
- removed link bh_palm_sensor_11_link
- removed link bh_palm_sensor_12_link
- removed link bh_palm_sensor_13_link
- removed link bh_palm_sensor_14_link
- removed link bh_palm_sensor_15_link
- removed link bh_palm_sensor_16_link
- removed link bh_palm_sensor_17_link
- removed link bh_palm_sensor_18_link
- removed link bh_palm_sensor_19_link
- removed link bh_palm_sensor_1_link
- removed link bh_palm_sensor_20_link
- removed link bh_palm_sensor_21_link
- removed link bh_palm_sensor_22_link
- removed link bh_palm_sensor_23_link
- removed link bh_palm_sensor_24_link
- removed link bh_palm_sensor_2_link
- removed link bh_palm_sensor_3_link
- removed link bh_palm_sensor_4_link
- removed link bh_palm_sensor_5_link
- removed link bh_palm_sensor_6_link
- removed link bh_palm_sensor_7_link
- removed link bh_palm_sensor_8_link
- removed link bh_palm_sensor_9_link
Joints:
- removed joint bh_link1_sensor10_joint
- removed joint bh_link1_sensor11_joint
- removed joint bh_link1_sensor12_joint
- removed joint bh_link1_sensor13_joint
- removed joint bh_link1_sensor14_joint
- removed joint bh_link1_sensor15_joint
- removed joint bh_link1_sensor16_joint
- removed joint bh_link1_sensor17_joint
- removed joint bh_link1_sensor18_joint
- removed joint bh_link1_sensor19_joint
- removed joint bh_link1_sensor1_joint
- removed joint bh_link1_sensor20_joint
- removed joint bh_link1_sensor21_joint
- removed joint bh_link1_sensor22_joint
- removed joint bh_link1_sensor23_joint
- removed joint bh_link1_sensor24_joint
- removed joint bh_link1_sensor2_joint
- removed joint bh_link1_sensor3_joint
- removed joint bh_link1_sensor4_joint
- removed joint bh_link1_sensor5_joint
- removed joint bh_link1_sensor6_joint
- removed joint bh_link1_sensor7_joint
- removed joint bh_link1_sensor8_joint
- removed joint bh_link1_sensor9_joint
- removed joint bh_link2_sensor10_joint
- removed joint bh_link2_sensor11_joint
- removed joint bh_link2_sensor12_joint
- removed joint bh_link2_sensor13_joint
- removed joint bh_link2_sensor14_joint
- removed joint bh_link2_sensor15_joint
- removed joint bh_link2_sensor16_joint
- removed joint bh_link2_sensor17_joint
- removed joint bh_link2_sensor18_joint
- removed joint bh_link2_sensor19_joint
- removed joint bh_link2_sensor1_joint
- removed joint bh_link2_sensor20_joint
- removed joint bh_link2_sensor21_joint
- removed joint bh_link2_sensor22_joint
- removed joint bh_link2_sensor23_joint
- removed joint bh_link2_sensor24_joint
- removed joint bh_link2_sensor2_joint
- removed joint bh_link2_sensor3_joint
- removed joint bh_link2_sensor4_joint
- removed joint bh_link2_sensor5_joint
- removed joint bh_link2_sensor6_joint
- removed joint bh_link2_sensor7_joint
- removed joint bh_link2_sensor8_joint
- removed joint bh_link2_sensor9_joint
- removed joint bh_link3_sensor10_joint
- removed joint bh_link3_sensor11_joint
- removed joint bh_link3_sensor12_joint
- removed joint bh_link3_sensor13_joint
- removed joint bh_link3_sensor14_joint
- removed joint bh_link3_sensor15_joint
- removed joint bh_link3_sensor16_joint
- removed joint bh_link3_sensor17_joint
- removed joint bh_link3_sensor18_joint
- removed joint bh_link3_sensor19_joint
- removed joint bh_link3_sensor1_joint
- removed joint bh_link3_sensor20_joint
- removed joint bh_link3_sensor21_joint
- removed joint bh_link3_sensor22_joint
- removed joint bh_link3_sensor23_joint
- removed joint bh_link3_sensor24_joint
- removed joint bh_link3_sensor2_joint
- removed joint bh_link3_sensor3_joint
- removed joint bh_link3_sensor4_joint
- removed joint bh_link3_sensor5_joint
- removed joint bh_link3_sensor6_joint
- removed joint bh_link3_sensor7_joint
- removed joint bh_link3_sensor8_joint
- removed joint bh_link3_sensor9_joint
- removed joint bh_palm_sensor10_joint
- removed joint bh_palm_sensor11_joint
- removed joint bh_palm_sensor12_joint
- removed joint bh_palm_sensor13_joint
- removed joint bh_palm_sensor14_joint
- removed joint bh_palm_sensor15_joint
- removed joint bh_palm_sensor16_joint
- removed joint bh_palm_sensor17_joint
- removed joint bh_palm_sensor18_joint
- removed joint bh_palm_sensor19_joint
- removed joint bh_palm_sensor1_joint
- removed joint bh_palm_sensor20_joint
- removed joint bh_palm_sensor21_joint
- removed joint bh_palm_sensor22_joint
- removed joint bh_palm_sensor23_joint
- removed joint bh_palm_sensor24_joint
- removed joint bh_palm_sensor2_joint
- removed joint bh_palm_sensor3_joint
- removed joint bh_palm_sensor4_joint
- removed joint bh_palm_sensor5_joint
- removed joint bh_palm_sensor6_joint
- removed joint bh_palm_sensor7_joint
- removed joint bh_palm_sensor8_joint
- removed joint bh_palm_sensor9_joint
